File: hardware/laser-range-finder.kicad_pcb (KiCad board)
At the start: 2 copper layers, 48.2 x 35.6 mm, 20 parts, among them K1 CONN_3, K2 CONN_3, P1 CON-SENSOR, U1 M24C64, U2 DRILL, U3 DRILL, U4 DRILL, U5 DRILL

Commit message: Add 3d information (final)
Parts:
- added REF**: LIDAR_v3, kicad-libraries:LIDAR_v3, B.Cu at (134.6, 103.7)
- C1, C2, C3, L1: footprint kicad-libraries:0603 -> kicad-libraries:C0603
- R1: footprint kicad-libraries:0603 -> kicad-libraries:R0603
Connections:
- RP1 pad 2: (no net) -> Net-(RP1-Pad2)
- RP1 pad 3: (no net) -> Net-(RP1-Pad3)
- U1 pad 7: (no net) -> Net-(U1-Pad7)
